Commit message: Update LRMate-200iD_convex.urdf
Modify the parameters of each pivot

File: urdf/LRMate-200iD_convex.urdf (robot description, URDF)
Before this commit: robot lrmate-200id, 8 links, 7 joints
Joints:
- joint J1: limit lower=-2.9671 upper=2.9671 effort=0 velocity=0 -> lower=-2.9671 upper=2.9671 effort=0 velocity=5.93
- joint J2: limit lower=-2.5307 upper=1.7453 effort=0 velocity=0 -> lower=-2.5307 upper=1.7453 effort=0 velocity=4.28
- joint J3: limit lower=-1.2217 upper=3.5779 effort=0 velocity=0 -> lower=-1.2217 upper=3.5779 effort=0 velocity=7.33
- joint J4: limit lower=-3.1416 upper=3.1416 effort=0 velocity=0 -> lower=-3.3161 upper=3.3161 effort=0 velocity=6.63
- joint J5: limit lower=-2.1817 upper=2.1817 effort=0 velocity=0 -> lower=-2.1817 upper=2.1817 effort=0 velocity=4.36
- joint J6: limit lower=0 upper=0 effort=0 velocity=0 -> lower=-6.2832 upper=6.2832 effort=0 velocity=12.57
